File: hardware/ARC86-512.kicad_sch (KiCad schematic)
At the start: 36 parts, among them J1 UART, J2 DISK1 IDE Interface, U1 80C88-2Z, U10 74HCT32, U11 AT28C256-15PU, U12 AS6C4008-55PCN, U13 82C59A, U14 74HCT138, U15 82C54, U16 82C55A, U17 SN75477P, U18 16C550D, U2 82C84A, U3 74HCT245, U4 74HCT573, U5 74HCT573, U6 74HCT573, U7 74HCT244, U8 74HCT04, U9 74HCT00, Y1 24MHz, Y2 3.072MHz

Commit message: REVC of schematic
Parts:
- LCD1: renamed from DS1; symbol Display_Character:HY1602E -> 8088_Library:HD44780
- U18: value 16C550D -> 16C550D (DIP-40); footprint Package_DIP:DIP-48_W15.24mm_LongPads -> Package_DIP:DIP-40_W15.24mm_LongPads; symbol 8088_Library:16C550D -> 8088_Library:16C550D_dip
Connections:
- net DATA0: now also U18.1 (D0); no longer U18.43 (D0)
- net DATA1: now also U18.2 (D1); no longer U18.44 (D1)
- net DATA2: now also U18.3 (D2); no longer U18.45 (D2)
- net DATA3: now also U18.4 (D3); no longer U18.46 (D3)
- net DATA4: now also U18.5 (D4); no longer U18.47 (D4)
- net DATA5: now also U18.6 (D5); no longer U18.2 (D5)
- net DATA6: now also U18.7 (D6); no longer U18.3 (D6)
- net DATA7: now also U18.8 (D7); no longer U18.4 (D7)
- net GND: now also U14.4 (~{E0}), U18.19 (WR), U18.22 (RD), U18.25 (~{ADS}); no longer LCD1.3 (VSS), R6.2, U14.5 (~{E1}), U14.6 (E2), U18.17 (WR), U18.18 (GND), U18.24 (~{ADS})
- net VCC: now also LCD1.15 (LEDA), U14.6 (E2), U18.12 (CS0), U18.13 (CS1), U18.40 (VCC), U2.4 (RDY1), U2.6 (RDY2); no longer LCD1.4 (VDD), U14.4 (~{E0}), U18.10 (CS1), U18.42 (VCC), U18.9 (CS0)
- net ~{IOR}: now also U18.21 (~{RD}); no longer U18.19 (~{RD})
- net ~{IOW}: now also U18.18 (~{WR}); no longer U18.16 (~{WR})
- net ~{SER1EN}: now also U18.14 (~{CS2}); no longer U18.11 (~{CS2})
- net M/~{IO}: now reaches U10.9, U8.6
- net M/~{IO}: now also U10.13, U14.5 (~{E1}); no longer U10.12
- net at U1.32 (~{RD}), U10.1: now also U8.5; no longer U10.13
- net at C2.1, R2.1, Y2.2: now also U18.16 (XIN); no longer U18.14 (XIN)
- net at LCD1.10 (DB3): now also U16.21 (PB3); no longer U16.19 (PB1)
- net at LCD1.11 (DB4): now also U16.22 (PB4); no longer U16.20 (PB2)
- net at LCD1.12 (DB5): now also U16.23 (PB5); no longer U16.21 (PB3)
- net at LCD1.13 (DB6): now also U16.24 (PB6); no longer U16.22 (PB4)
- net at LCD1.14 (DB7): now also U16.25 (PB7); no longer U16.23 (PB5)
- net at LCD1.16 (LEDK): now also R6.2; no longer U16.25 (PB7)
- net at R5.2: now also LCD1.3 (Vo); no longer LCD1.5 (Vo)
- net at U16.16 (PC2): now also LCD1.4 (RS); no longer LCD1.6 (RS)
- net at U16.15 (PC1): now also LCD1.5 (R/~{W}); no longer LCD1.7 (R/~{W})
- net at U16.14 (PC0): now also LCD1.6 (E); no longer LCD1.8 (E)
- net at U16.18 (PB0): now also LCD1.7 (DB0); no longer LCD1.9 (DB0)
- net at U1.28 (IO/~{M}), U10.2, U10.4: now also U10.12; no longer U8.5
- net at U18.15 (~{BAUDOUT}): now also U18.9 (RCLK); no longer R3.2
- net at J1.3 (Pin_3): now also U18.10 (SIN); no longer U18.7 (SIN)
- net at J1.2 (Pin_2): now also U18.11 (SOUT); no longer U18.8 (SOUT)
- net at U1.9 (AD7), U3.2 (A0), U6.2 (D0): now also U13.4 (D7); no longer U13.11 (D0)
- net at U1.10 (AD6), U3.3 (A1), U6.3 (D1): now also U13.5 (D6); no longer U13.10 (D1)
- net at U1.11 (AD5), U3.4 (A2), U6.4 (D2): now also U13.6 (D5); no longer U13.9 (D2)
- net at U1.12 (AD4), U3.5 (A3), U6.5 (D3): now also U13.7 (D4); no longer U13.8 (D3)
- net at U1.13 (AD3), U3.6 (A4), U6.6 (D4): now also U13.8 (D3); no longer U13.7 (D4)
- net at U1.14 (AD2), U3.7 (A5), U6.7 (D5): now also U13.9 (D2); no longer U13.6 (D5)
- net at U1.15 (AD1), U3.8 (A6), U6.8 (D6): now also U13.10 (D1); no longer U13.5 (D6)
- net at U1.16 (AD0), U3.9 (A7), U6.9 (D7): now also U13.11 (D0); no longer U13.4 (D7)
- new net: LCD1.8 (DB1), U16.19 (PB1)
- new net: LCD1.9 (DB2), U16.20 (PB2)
- new net: R3.2, U18.17 (XOUT)
- no-connect marks 53 -> 51
Other:
- moved on the sheet: U8C

Commit message: Rev D of schematic
Parts:
- renumbered R7 to R5
Connections:
- net GND: no longer J2.10 (Pin_10), J2.12 (Pin_12), J2.14 (Pin_14), J2.16 (Pin_16), J2.18 (Pin_18), J2.2 (Pin_2), J2.22 (Pin_22), J2.24 (Pin_24), J2.26 (Pin_26), J2.30 (Pin_30), J2.4 (Pin_4), J2.6 (Pin_6), J2.8 (Pin_8)
- net IRQ3: now also U18.30 (INTR)
- net IRQ4: no longer U18.30 (INTR)
- net IRQ5: now also J2.31 (Pin_31)
- net VCC: now also J2.20 (Pin_20)
- no-connect marks 51 -> 62
Other:
- note added: "R1 - Brown-Black-Orange R2 - Brown-Black-Green R3 - Brown-Green-Red R4 - Yellow-Purple-Red R5 - Orange-Orange-Black C1 - 106 C2 - 22 C3 - 47 C4 - 103"
- note added: "Resistor & Capacitor Markings"
